Commit message: corrected the topics and added the plugins for sensors and tested them in simulation and updated generate assets and xacro

File: src/wafl_simulation/urdf/wafl_gz_plugins.xacro (robot description, xacro)
@@ -5,45 +5,85 @@
   Include from the robot xacro with:
       <xacro:include filename="$(find wafl_simulation)/urdf/wafl_gz_plugins.xacro"/>
-  The robot URDF MUST provide (names are what config/ros_gz_bridge.yaml relies on):
-      joints : left_wheel_joint, right_wheel_joint (continuous, rotate about the axle),
-               caster_joint (revolute, +-80 deg), fork_joint (prismatic, up = +)
-      links  : laser_link, camera_link (x forward), imu_link
+  CONTRACT (README sec. 6 / D23). The robot URDF MUST provide these joints (names are what
+  config/ros_gz_bridge.yaml relies on) - geometry, origins and axes are NOT used here:
+      front_left_steer_joint, front_right_steer_joint  revolute, axis +z   (front pair, steered together)
+      caster_joint                                     revolute, axis +z   (REAR wheel steering)
+      front_left_wheel_joint, front_right_wheel_joint  continuous          (the only driven wheels)
+      caster_wheel_joint                               continuous, PASSIVE (no plugin, must roll freely)
+      fork_joint                                       prismatic, up = +
+  links : base_footprint (origin = midpoint of the front drive axle), laser_link, camera_link (x forward),
+          imu_link
   Gazebo model name MUST be "wafl" (gazebo.launch.py spawns with -name wafl).
   Design rules taken from the README:
-    * DiffDrive listens on /model/wafl/cmd_vel  <- ros /cmd_vel_out (arbitrated), NEVER raw /cmd_vel.
-    * DiffDrive TF is sent to an UNBRIDGED topic: the EKF is the only odom->base_footprint publisher.
-    * Caster = joint position controller (radians) on /model/wafl/joint/caster_joint/cmd_pos.
-    * Fork   = joint velocity controller on /model/wafl/joint/fork_joint/cmd_vel.
+    * NO DiffDrive (it cannot model steered wheels) and NO /cmd_vel_out: Gazebo only receives per-joint commands,
+      published by base_controller AFTER arbitration. Raw /cmd_vel is never read.
+    * Odometry = OdometryPublisher (ground truth). Its TF goes to an UNBRIDGED topic: the EKF is the only
+      odom->base_footprint publisher.
+    * Both front steering joints subscribe to the SAME gz topic, so they stay parallel like the real chain.
+    * Wheel mode (kinematic | force) and every gain live in config/sim_controllers.yaml - no regeneration needed.
 -->
 <robot xmlns:xacro="http://www.ros.org/wiki/xacro">
-  <xacro:arg name="wheel_radius" default="0.1"/>
-  <xacro:arg name="track_width"  default="0.3395"/>
+  <xacro:arg name="sim_controllers_yaml" default="$(find wafl_simulation)/config/sim_controllers.yaml"/>
+  <xacro:property name="sim_cfg_file" value="$(arg sim_controllers_yaml)"/>
+  <xacro:property name="sim_cfg" value="${xacro.load_yaml(sim_cfg_file)}"/>
+  <xacro:property name="wheel_force" value="${sim_cfg['wheel_drive']['mode'] == 'force'}"/>
+  <!-- Front drive wheel: velocity command in rad/s. kinematic = joint velocity is set directly;
+       force = PID applies torque (use_force_commands). -->
+  <xacro:macro name="wheel_velocity_controller" params="joint">
+    <gazebo>
+      <plugin filename="gz-sim-joint-controller-system" name="gz::sim::systems::JointController">
+        <joint_name>${joint}</joint_name>
+        <topic>/model/wafl/joint/${joint}/cmd_vel</topic>
+        <initial_velocity>0.0</initial_velocity>
+        <xacro:if value="${wheel_force}">
+          <use_force_commands>true</use_force_commands>
+          <p_gain>${sim_cfg['wheel_drive']['p_gain']}</p_gain>
+          <i_gain>${sim_cfg['wheel_drive']['i_gain']}</i_gain>
+          <d_gain>${sim_cfg['wheel_drive']['d_gain']}</d_gain>
+          <i_max>${sim_cfg['wheel_drive']['i_max']}</i_max>
+          <i_min>${sim_cfg['wheel_drive']['i_min']}</i_min>
+          <cmd_max>${sim_cfg['wheel_drive']['cmd_max']}</cmd_max>
+          <cmd_min>${sim_cfg['wheel_drive']['cmd_min']}</cmd_min>
+        </xacro:if>
+      </plugin>
+    </gazebo>
+  </xacro:macro>
+  <!-- Steering joint: position command in radians (a stepper on the real robot). -->
+  <xacro:macro name="steer_position_controller" params="joint topic">
+    <gazebo>
+      <plugin filename="gz-sim-joint-position-controller-system" name="gz::sim::systems::JointPositionController">
+        <joint_name>${joint}</joint_name>
+        <topic>${topic}</topic>
+        <p_gain>${sim_cfg['steering']['p_gain']}</p_gain>
+        <i_gain>${sim_cfg['steering']['i_gain']}</i_gain>
+        <d_gain>${sim_cfg['steering']['d_gain']}</d_gain>
+        <i_max>${sim_cfg['steering']['i_max']}</i_max>
+        <i_min>${sim_cfg['steering']['i_min']}</i_min>
+        <cmd_max>${sim_cfg['steering']['cmd_max']}</cmd_max>
+        <cmd_min>${sim_cfg['steering']['cmd_min']}</cmd_min>
+      </plugin>
+    </gazebo>
+  </xacro:macro>
+  <xacro:wheel_velocity_controller joint="front_left_wheel_joint"/>
+  <xacro:wheel_velocity_controller joint="front_right_wheel_joint"/>
+  <!-- both front steering joints share ONE gz topic -> always parallel (same as the real chain/sprocket) -->
+  <xacro:steer_position_controller joint="front_left_steer_joint"  topic="/model/wafl/front_steer/cmd_pos"/>
+  <xacro:steer_position_controller joint="front_right_steer_joint" topic="/model/wafl/front_steer/cmd_pos"/>
+  <!-- rear wheel steering; topic set explicitly (the default would include the axis index, /0/cmd_pos) -->
+  <xacro:steer_position_controller joint="caster_joint" topic="/model/wafl/joint/caster_joint/cmd_pos"/>
   <gazebo>
-    <plugin filename="gz-sim-diff-drive-system" name="gz::sim::systems::DiffDrive">
-      <left_joint>leftwheel</left_joint>
-      <right_joint>rightwheel</right_joint>
-      <wheel_separation>$(arg track_width)</wheel_separation>
-      <wheel_radius>$(arg wheel_radius)</wheel_radius>
-      <topic>/model/wafl/cmd_vel</topic>
+    <!-- ground-truth odometry. Output topic is bridged to /odom; the TF it also emits goes to a dead-end topic. -->
+    <plugin filename="gz-sim-odometry-publisher-system" name="gz::sim::systems::OdometryPublisher">
+      <odom_frame>odom</odom_frame>
+      <robot_base_frame>base_footprint</robot_base_frame>
       <odom_topic>/model/wafl/odometry</odom_topic>
       <tf_topic>/model/wafl/tf_unused_ekf_owns_odom_tf</tf_topic>
-      <frame_id>odom</frame_id>
-      <child_frame_id>base_footprint</child_frame_id>
       <odom_publish_frequency>50</odom_publish_frequency>
-      <max_linear_velocity>1.0</max_linear_velocity>
-      <min_linear_velocity>-1.0</min_linear_velocity>
-      <max_angular_velocity>1.5</max_angular_velocity>
-      <min_angular_velocity>-1.5</min_angular_velocity>
+      <dimensions>2</dimensions>
     </plugin>
-    <plugin filename="gz-sim-joint-position-controller-system" name="gz::sim::systems::JointPositionController">
-      <joint_name>castorjoint</joint_name>
-      <topic>/model/wafl/joint/caster_joint/cmd_pos</topic>
-      <p_gain>8.0</p_gain>
-      <i_gain>0.1</i_gain>
-      <d_gain>0.4</d_gain>
-      <i_max>1.0</i_max>
-      <i_min>-1.0</i_min>
-      <cmd_max>20.0</cmd_max>
-      <cmd_min>-20.0</cmd_min>
+    <plugin filename="gz-sim-joint-controller-system" name="gz::sim::systems::JointController">
+      <joint_name>fork_joint</joint_name>
+      <topic>/model/wafl/joint/fork_joint/cmd_vel</topic>
+      <initial_velocity>0.0</initial_velocity>
     </plugin>
     <plugin filename="gz-sim-joint-state-publisher-system" name="gz::sim::systems::JointStatePublisher"/>
